Commit message: Rework the description palette for legibility in RViz
The arm was graphite, 0.18 grey. RViz lights a dark model badly: against the
default dark background the shading collapses and the five links read as one
silhouette with no visible edges between them, which makes it impossible to
tell by eye whether a joint origin is where it should be.

The palette now separates by role rather than by taste. Printed structure is
light grey, brackets and fasteners a shade down so a joint reads against the
link it sits on, and the tool body is the darkest thing in the scene so the
placeholder is never mistaken for measured hardware. The accent red is kept
for the needle and anything else that has to be found at a glance.

tattotronix_graphite is renamed to tattotronix_shell; the name described a
colour, and what callers actually select is a role.

File: src/tattotronix_description/urdf/materials.xacro (robot description, xacro)
@@ -2,5 +2,5 @@
 <robot xmlns:xacro="http://www.ros.org/wiki/xacro">
   <!--
-    Shared RViz colours.
+    Shared colours.
     Wrapped in a macro rather than declared at file scope on purpose. Both the
     arm and the tool macros include this file, and xacro does not deduplicate
@@ -8,15 +8,23 @@
     URDF parser rejects a duplicate material name. The macro is expanded once,
     by the top-level description.
+    The arm is light grey because RViz lights a dark model badly: on the dark
+    background the shading collapses and the whole arm reads as one silhouette
+    with no edges. Grey keeps the links separable. The pen stays dark so it is
+    obvious which part of the model is hardware and which is the placeholder.
   -->
   <xacro:macro name="tattotronix_materials">
-    <material name="tattotronix_graphite">
-      <color rgba="0.18 0.18 0.20 1.0"/>
+    <!-- Printed structure. -->
+    <material name="tattotronix_shell">
+      <color rgba="0.78 0.79 0.81 1.0"/>
     </material>
+    <!-- Brackets and fasteners, a shade down so joints read against links. -->
     <material name="tattotronix_steel">
-      <color rgba="0.70 0.72 0.75 1.0"/>
+      <color rgba="0.55 0.57 0.61 1.0"/>
     </material>
+    <!-- Tool body. Deliberately the darkest thing in the scene. -->
     <material name="tattotronix_ink">
-      <color rgba="0.05 0.05 0.07 1.0"/>
+      <color rgba="0.13 0.13 0.16 1.0"/>
     </material>
+    <!-- Needle, and anything else that has to be found at a glance. -->
     <material name="tattotronix_accent">
       <color rgba="0.85 0.25 0.20 1.0"/>
