Commit message: Reduce the tattoo pen to the simplest shape that can carry a TCP
The pen was built from primitives sized to a catalogue rotary machine: a
105 mm barrel of 25 mm diameter, a 30 mm tapered grip and a protruding
needle. None of it was measured. The pen has not been built, so every one of
those numbers was invention with the shape of hardware, and a detailed
placeholder is worse than an obvious one because it invites people to measure
off it and to plan reach and clearance against dimensions nobody chose.

It is now a single cylinder, 45 mm long and 3 mm in radius, parameterised on
the macro so both numbers change in one place. What the description has to get
right is the axis and the tip, since those are what tattoo paths are planned
against, and both survive the simplification.

The inertia is kept as a real cylinder tensor rather than a guess, so the link
stays valid under an effort-aware controller.

File: src/tattotronix_description/urdf/tattoo_tool.xacro (robot description, xacro)
@@ -1,98 +1,49 @@
 <?xml version="1.0"?>
 <robot xmlns:xacro="http://www.ros.org/wiki/xacro">
-  <xacro:include filename="$(find tattotronix_description)/urdf/inertial_macros.xacro"/>
   <xacro:include filename="$(find tattotronix_description)/urdf/materials.xacro"/>
   <!--
-    Rotary tattoo pen mounted on tool0.
-    There is no CAD for the pen yet, so it is built from primitives sized to a
-    standard rotary machine: a 105 mm barrel of 25 mm diameter, a 30 mm tapered
-    grip, and the needle protruding past it. The frame that matters downstream
-    is tattoo_tcp, which sits at the needle tip with +z pointing along the
-    needle, into the skin. Every tattoo path is planned for that frame, so when
-    the real pen is measured only the offsets in this file change.
+    Tattoo pen: one thin cylinder along the tool axis, and the frame at its tip.
+    Deliberately the simplest shape that can carry a TCP. The pen has not been
+    built, so any detail here would be invention dressed up as hardware, and a
+    detailed placeholder is worse than an obvious one: it invites people to
+    measure off it. What this has to get right is the axis and the tip, because
+    those are what tattoo paths are planned against, and both are replaceable
+    by editing two numbers when the real pen is measured.
+    The frame to plan in is tattoo_tcp, at the tip, +z pointing along the pen
+    and into the work.
   -->
-  <xacro:macro name="tattoo_tool" params="parent">
-    <xacro:property name="barrel_length" value="0.105"/>
-    <xacro:property name="barrel_radius" value="0.0125"/>
-    <xacro:property name="grip_length" value="0.030"/>
-    <xacro:property name="grip_radius" value="0.006"/>
-    <xacro:property name="needle_length" value="0.008"/>
-    <xacro:property name="needle_radius" value="0.0006"/>
+  <xacro:macro name="tattoo_tool" params="parent length:=0.045 radius:=0.003">
     <joint name="tool0_to_tattoo_pen" type="fixed">
       <parent link="${parent}"/>
       <child link="tattoo_pen_link"/>
-      <!-- No rotation. tool0 already defines +z as the tool axis, which is the
-           SG90 output shaft, so the pen inherits the alignment instead of
-           re-deriving it and drifting away from the flange. -->
+      <!-- No rotation: tool0 already defines +z as the tool axis. -->
       <origin xyz="0 0 0" rpy="0 0 0"/>
     </joint>
     <link name="tattoo_pen_link">
       <visual>
-        <origin xyz="0 0 ${barrel_length/2}" rpy="0 0 0"/>
+        <origin xyz="0 0 ${length/2}" rpy="0 0 0"/>
         <geometry>
-          <cylinder radius="${barrel_radius}" length="${barrel_length}"/>
+          <cylinder radius="${radius}" length="${length}"/>
         </geometry>
         <material name="tattotronix_ink"/>
       </visual>
       <collision>
-        <origin xyz="0 0 ${barrel_length/2}" rpy="0 0 0"/>
+        <origin xyz="0 0 ${length/2}" rpy="0 0 0"/>
         <geometry>
-          <cylinder radius="${barrel_radius}" length="${barrel_length}"/>
+          <cylinder radius="${radius}" length="${length}"/>
         </geometry>
       </collision>
-      <xacro:inertial_cylinder mass="0.150" radius="${barrel_radius}" length="${barrel_length}">
-        <origin xyz="0 0 ${barrel_length/2}" rpy="0 0 0"/>
-      </xacro:inertial_cylinder>
-    </link>
-    <joint name="tattoo_pen_to_grip" type="fixed">
-      <parent link="tattoo_pen_link"/>
-      <child link="tattoo_grip_link"/>
-      <origin xyz="0 0 ${barrel_length}" rpy="0 0 0"/>
-    </joint>
-    <link name="tattoo_grip_link">
-      <visual>
-        <origin xyz="0 0 ${grip_length/2}" rpy="0 0 0"/>
-        <geometry>
-          <cylinder radius="${grip_radius}" length="${grip_length}"/>
-        </geometry>
-        <material name="tattotronix_steel"/>
-      </visual>
-      <collision>
-        <origin xyz="0 0 ${grip_length/2}" rpy="0 0 0"/>
-        <geometry>
-          <cylinder radius="${grip_radius}" length="${grip_length}"/>
-        </geometry>
-      </collision>
-      <xacro:inertial_cylinder mass="0.030" radius="${grip_radius}" length="${grip_length}">
-        <origin xyz="0 0 ${grip_length/2}" rpy="0 0 0"/>
-      </xacro:inertial_cylinder>
-    </link>
-    <!-- The needle is visual only. Giving it collision geometry would make the
-         contact solver fight a 0.6 mm cylinder every step for no benefit; skin
-         contact is modelled at the TCP, not by the mesh. -->
-    <joint name="tattoo_grip_to_needle" type="fixed">
-      <parent link="tattoo_grip_link"/>
-      <child link="tattoo_needle_link"/>
-      <origin xyz="0 0 ${grip_length}" rpy="0 0 0"/>
-    </joint>
-    <link name="tattoo_needle_link">
-      <visual>
-        <origin xyz="0 0 ${needle_length/2}" rpy="0 0 0"/>
-        <geometry>
-          <cylinder radius="${needle_radius}" length="${needle_length}"/>
-        </geometry>
-        <material name="tattotronix_accent"/>
-      </visual>
       <inertial>
-        <origin xyz="0 0 ${needle_length/2}" rpy="0 0 0"/>
-        <mass value="0.001"/>
-        <inertia ixx="1e-8" ixy="0.0" ixz="0.0" iyy="1e-8" iyz="0.0" izz="1e-8"/>
+        <origin xyz="0 0 ${length/2}" rpy="0 0 0"/>
+        <mass value="0.020"/>
+        <inertia ixx="${0.020 * (3.0*radius*radius + length*length) / 12.0}" ixy="0.0" ixz="0.0"
+                 iyy="${0.020 * (3.0*radius*radius + length*length) / 12.0}" iyz="0.0"
+                 izz="${0.020 * radius * radius / 2.0}"/>
       </inertial>
     </link>
-    <!-- Tool centre point: needle tip, +z along the needle. -->
-    <joint name="tattoo_needle_to_tcp" type="fixed">
-      <parent link="tattoo_needle_link"/>
+    <joint name="tattoo_pen_to_tcp" type="fixed">
+      <parent link="tattoo_pen_link"/>
       <child link="tattoo_tcp"/>
-      <origin xyz="0 0 ${needle_length}" rpy="0 0 0"/>
+      <origin xyz="0 0 ${length}" rpy="0 0 0"/>
     </joint>
     <link name="tattoo_tcp"/>

Commit message: Give the tattoo pen a pointed tip
A needle that ends in a flat disc reads wrong in RViz and Gazebo. URDF has
no cone primitive, so the tip is a generated mesh: make_pen_tip.py writes
it parametrically rather than leaving a binary blob in the tree that
nobody can regenerate or check.

Cosmetic only, and deliberately kept away from anything measured. The
barrel shortens by the taper and the cone fills it, so total length and
`tattoo_tcp` are untouched: forward kinematics still puts the tip at
258.96, -9.44, 245.58 mm at the zero pose, which is the value verified
against live TF. Collision stays the full cylinder, which is conservative
and keeps a sharp cone out of the contact solver.

The mesh is written in millimetres and scaled 0.001, unlike the exported
CAD meshes which are in centimetres and scaled 0.01.

File: src/tattotronix_description/urdf/tattoo_tool.xacro (robot description, xacro)
@@ -3,5 +3,6 @@
   <xacro:include filename="$(find tattotronix_description)/urdf/materials.xacro"/>
   <!--
-    Tattoo pen: one thin cylinder along the tool axis, and the frame at its tip.
+    Tattoo pen: a thin barrel along the tool axis with a conical tip, and the
+    frame at that tip.
     Deliberately the simplest shape that can carry a TCP. The pen has not been
     built, so any detail here would be invention dressed up as hardware, and a
@@ -13,5 +14,5 @@
     and into the work.
   -->
-  <xacro:macro name="tattoo_tool" params="parent length:=0.045 radius:=0.003">
+  <xacro:macro name="tattoo_tool" params="parent length:=0.045 radius:=0.003 taper:=0.008">
     <joint name="tool0_to_tattoo_pen" type="fixed">
       <parent link="${parent}"/>
@@ -21,11 +22,32 @@
     </joint>
     <link name="tattoo_pen_link">
+      <!-- Barrel: full length minus the taper. -->
       <visual>
-        <origin xyz="0 0 ${length/2}" rpy="0 0 0"/>
+        <origin xyz="0 0 ${(length - taper)/2}" rpy="0 0 0"/>
         <geometry>
-          <cylinder radius="${radius}" length="${length}"/>
+          <cylinder radius="${radius}" length="${length - taper}"/>
         </geometry>
         <material name="tattotronix_ink"/>
       </visual>
+      <!--
+        Tip: a cone, because URDF has no cone primitive and a flat disc at the
+        end of a needle reads wrong. The mesh is generated by
+        docs/scripts/make_pen_tip.py and written in millimetres, hence the 0.001
+        scale; the exported CAD meshes are in centimetres and carry 0.01
+        instead. Its apex lands exactly on tattoo_tcp - the tip has not moved.
+      -->
+      <visual>
+        <origin xyz="0 0 ${length - taper}" rpy="0 0 0"/>
+        <geometry>
+          <mesh filename="package://tattotronix_description/meshes/visual/tattoo_pen_tip.stl"
+                scale="0.001 0.001 0.001"/>
+        </geometry>
+        <material name="tattotronix_ink"/>
+      </visual>
+      <!--
+        Collision stays the full cylinder. It is conservative, it is what a
+        collision check should use, and it keeps the tip out of the contact
+        solver where a sharp cone would only make it brittle.
+      -->
       <collision>
         <origin xyz="0 0 ${length/2}" rpy="0 0 0"/>
