Commit message: Make the description parse: legal XML comments and one materials block
Two defects that only surface once xacro and the URDF parser actually run
over the file:

The joint section headers padded their comments out to the right margin with
runs of hyphens. XML forbids a double hyphen inside a comment, so xacro
rejected the file before it reached any macro.

materials.xacro declared its colours at file scope and is included by both
arm_macro.xacro and tattoo_tool.xacro. xacro does not deduplicate includes,
so the colours were emitted twice and urdf rejected the duplicate name. The
colours now live in a macro the top-level description expands exactly once,
which keeps each macro free to declare what it needs.

Verified with check_urdf across the four configurations that matter:
hardware none, mock and gz, with and without the tattoo pen, and with the
world anchor disabled. The tree resolves world -> base_link through the five
axes to tattoo_tcp.

File: src/tattotronix_description/urdf/arm_macro.xacro (robot description, xacro)
@@ -45,5 +45,5 @@
   </xacro:macro>
   <xacro:macro name="tattotronix_arm" params="parent *origin">
-    <!-- base ---------------------------------------------------------------->
+    <!-- base -->
     <joint name="base_mount" type="fixed">
       <parent link="${parent}"/>
@@ -54,5 +54,5 @@
         cx="-0.03125" cy="-0.0013" cz="0.02435"
         sx="0.1575" sy="0.0950" sz="0.0485"/>
-    <!-- joint 1: base yaw ---------------------------------------------------->
+    <!-- joint 1: base yaw -->
     <joint name="joint_1" type="revolute">
       <parent link="base_link"/>
@@ -66,5 +66,5 @@
         cx="0.00075" cy="0.0" cz="0.03455"
         sx="0.0945" sy="0.1251" sz="0.0667"/>
-    <!-- joint 2: shoulder pitch ---------------------------------------------->
+    <!-- joint 2: shoulder pitch -->
     <joint name="joint_2" type="revolute">
       <parent link="shoulder_link"/>
@@ -78,5 +78,5 @@
         cx="0.0" cy="-0.00255" cz="0.0567"
         sx="0.0390" sy="0.0461" sz="0.1522"/>
-    <!-- joint 3: elbow pitch ------------------------------------------------->
+    <!-- joint 3: elbow pitch -->
     <joint name="joint_3" type="revolute">
       <parent link="upper_arm_link"/>
@@ -90,5 +90,5 @@
         cx="-0.0109" cy="-0.0230" cz="0.0330"
         sx="0.0670" sy="0.0460" sz="0.0910"/>
-    <!-- joint 4: wrist roll -------------------------------------------------->
+    <!-- joint 4: wrist roll -->
     <joint name="joint_4" type="revolute">
       <parent link="forearm_link"/>
@@ -102,5 +102,5 @@
         cx="0.08525" cy="0.00915" cz="-0.00005"
         sx="0.1705" sy="0.0569" sz="0.0364"/>
-    <!-- joint 5: wrist pitch ------------------------------------------------->
+    <!-- joint 5: wrist pitch -->
     <joint name="joint_5" type="revolute">
       <parent link="wrist_link"/>
@@ -114,5 +114,5 @@
         cx="0.0076" cy="-0.01155" cz="-0.0037"
         sx="0.0492" sy="0.0231" sz="0.0414"/>
-    <!-- tool flange ----------------------------------------------------------
+    <!-- tool flange.
          tool0 is the industrial flange frame every end effector attaches to.
          It sits on the far face of the tool mount mesh, centred on the mount

File: src/tattotronix_description/urdf/materials.xacro (robot description, xacro)
@@ -1,15 +1,25 @@
 <?xml version="1.0"?>
 <robot xmlns:xacro="http://www.ros.org/wiki/xacro">
-  <material name="tattotronix_graphite">
-    <color rgba="0.18 0.18 0.20 1.0"/>
-  </material>
-  <material name="tattotronix_steel">
-    <color rgba="0.70 0.72 0.75 1.0"/>
-  </material>
-  <material name="tattotronix_ink">
-    <color rgba="0.05 0.05 0.07 1.0"/>
-  </material>
-  <material name="tattotronix_accent">
-    <color rgba="0.85 0.25 0.20 1.0"/>
-  </material>
+  <!--
+    Shared RViz colours.
+    Wrapped in a macro rather than declared at file scope on purpose. Both the
+    arm and the tool macros include this file, and xacro does not deduplicate
+    includes, so file-scope <material> elements would be emitted twice and the
+    URDF parser rejects a duplicate material name. The macro is expanded once,
+    by the top-level description.
+  -->
+  <xacro:macro name="tattotronix_materials">
+    <material name="tattotronix_graphite">
+      <color rgba="0.18 0.18 0.20 1.0"/>
+    </material>
+    <material name="tattotronix_steel">
+      <color rgba="0.70 0.72 0.75 1.0"/>
+    </material>
+    <material name="tattotronix_ink">
+      <color rgba="0.05 0.05 0.07 1.0"/>
+    </material>
+    <material name="tattotronix_accent">
+      <color rgba="0.85 0.25 0.20 1.0"/>
+    </material>
+  </xacro:macro>
 </robot>

File: src/tattotronix_description/urdf/tattotronix.urdf.xacro (robot description, xacro)
@@ -24,8 +24,10 @@
   <xacro:property name="tool" value="$(arg tool)"/>
   <xacro:property name="use_world_link" value="$(arg use_world_link)"/>
+  <xacro:include filename="$(find tattotronix_description)/urdf/materials.xacro"/>
   <xacro:include filename="$(find tattotronix_description)/urdf/arm_macro.xacro"/>
   <xacro:include filename="$(find tattotronix_description)/urdf/tattoo_tool.xacro"/>
   <xacro:include filename="$(find tattotronix_description)/urdf/tattotronix.ros2_control.xacro"/>
   <xacro:include filename="$(find tattotronix_description)/urdf/tattotronix.gazebo.xacro"/>
+  <xacro:tattotronix_materials/>
   <!-- Anchor. The ROS 1 description referenced a world link it never declared,
        so the tree had a dangling parent and only loaded because nothing

Commit message: Align the tattoo pen with the SG90 output shaft and restore the bracket
The pen was mounted along the flange +x axis, across the servo shaft instead
of along it, which is why it read as bolted on at an angle.

The bracket mesh gives the axis away. Its two clamp faces sit at y = -6.0 mm
and y = -18.0 mm, a 12.0 mm gap, which is the body width of an SG90, and they
share a centroid at x = 4.5 mm, z = -3.0 mm. That fixes the shaft line. tool0
now sits where that line leaves the outer face of the bracket at y = -23.1 mm,
with +z along the shaft and pointing away from the arm, so a tool mounts with
no rotation of its own and inherits the alignment rather than re-deriving it.

The bracket mesh comes back with the correction, since what made it look wrong
was the pen crossing it rather than the part itself.

The servo is a continuous-rotation conversion and what it drives is not
decided, so the tool joint stays fixed. The axis is recorded in the geometry
and nothing is actuated on a guess.

Offsets are read off the mesh, not off CAD datums; expect a millimetre or two
of correction once the bracket is measured.

File: src/tattotronix_description/urdf/arm_macro.xacro (robot description, xacro)
@@ -111,16 +111,29 @@
       <dynamics damping="${joint_damping}" friction="${joint_friction}"/>
     </joint>
+    <!-- Tool mount: a bracket carrying a continuous-rotation SG90.
+         The mesh is a clamp whose two arms face each other across a 12.0 mm
+         gap, which is the body width of an SG90, so the servo sits between
+         them with its output shaft on the bracket's y axis. What that servo
+         ends up driving is not settled, so nothing here actuates: the tool
+         attaches through a fixed joint and the axis is recorded, not moved. -->
     <xacro:tattotronix_link name="tool_mount_link" mass="0.15"
         cx="0.0076" cy="-0.01155" cz="-0.0037"
         sx="0.0492" sy="0.0231" sz="0.0414"/>
     <!-- tool flange.
-         tool0 is the industrial flange frame every end effector attaches to.
-         It sits on the far face of the tool mount mesh, centred on the mount
-         in y and z. Derived from the mesh bounding box, not from CAD datums,
-         so treat it as accurate to a couple of millimetres until confirmed. -->
+         tool0 is the frame every end effector attaches to, and its +z axis is
+         the tool axis, so a tool mounts with no rotation of its own.
+         It is placed on the servo axis rather than guessed: the bracket's two
+         clamp faces lie at y = -6.0 mm and y = -18.0 mm and share a centroid
+         at x = 4.5 mm, z = -3.0 mm, which fixes the shaft line. tool0 sits
+         where that line leaves the outer face of the bracket, y = -23.1 mm,
+         with +z pointing away from the arm. This is why the pen used to look
+         wrong: it was mounted along +x, across the servo shaft instead of
+         along it.
+         Read off the mesh, not off CAD datums. Expect it to move by a
+         millimetre or two once the bracket is measured. -->
     <joint name="tool_mount_to_tool0" type="fixed">
       <parent link="tool_mount_link"/>
       <child link="tool0"/>
-      <origin xyz="0.0322 -0.01155 0.0" rpy="0 0 0"/>
+      <origin xyz="0.0045 -0.0231 -0.0030" rpy="${pi/2} 0 0"/>
     </joint>
     <link name="tool0"/>

File: src/tattotronix_description/urdf/tattoo_tool.xacro (robot description, xacro)
@@ -22,6 +22,8 @@
       <parent link="${parent}"/>
       <child link="tattoo_pen_link"/>
-      <!-- The pen points along the flange +x axis, barrel base on the flange. -->
-      <origin xyz="0 0 0" rpy="0 ${pi/2} 0"/>
+      <!-- No rotation. tool0 already defines +z as the tool axis, which is the
+           SG90 output shaft, so the pen inherits the alignment instead of
+           re-deriving it and drifting away from the flange. -->
+      <origin xyz="0 0 0" rpy="0 0 0"/>
     </joint>
     <link name="tattoo_pen_link">

File: src/tattotronix_description/urdf/tattotronix.urdf.xacro (robot description, xacro)
@@ -10,12 +10,10 @@
                         display.launch.py wants: a description RViz can render
                         with joint_state_publisher_gui and no controller stack.
-      tool              none | tattoo
-                        Defaults to none, which is the CAD and nothing else.
-                        'tattoo' adds the placeholder pen described in
-                        tattoo_tool.xacro: primitives sized to a standard
-                        rotary machine, not measured hardware. It exists so
-                        that the TCP the paths are planned for has a frame,
-                        and it is opt-in so that nothing invented is ever
-                        mistaken for the real robot.
+      tool              tattoo | none
+                        The pen in tattoo_tool.xacro is primitives sized to a
+                        catalogue rotary machine, not measured hardware. It is
+                        the default because the TCP the tattoo paths are
+                        planned for has to exist; 'none' strips it back to the
+                        exported CAD when the question is about the arm.
       controllers_file  absolute path to the controller manager YAML, read by
                         the Gazebo plugin. Only consulted when hardware=gz.
@@ -25,5 +23,5 @@
   -->
   <xacro:arg name="hardware" default="none"/>
-  <xacro:arg name="tool" default="none"/>
+  <xacro:arg name="tool" default="tattoo"/>
   <xacro:arg name="controllers_file" default=""/>
   <xacro:arg name="use_world_link" default="true"/>

Commit message: Put every collision mesh in the frame of the visual it belongs to
The CAD was exported twice, STL for the visuals and COLLADA for the collision
shapes, and the two runs did not agree on axes. Each DAE declares Z_UP while
its coordinates are Y-up, so five of the six links collided with a shape
rotated 90 degrees about X relative to what was drawn; the wrist was rotated
about Y instead, and three carried a translation on top of that. A URDF never
checks that a link's two geometries describe the same object, so none of this
was reported anywhere. It would have shown up as an arm that pushes objects it
is not touching and passes through ones it is.

The meshes themselves were never in doubt: every DAE has the same triangle
count and the same surface area as its STL, to 0.01 cm2, so the pair differ by
a rigid transform and nothing else. tools/align_collision_meshes.py recovers
that transform, verifying a candidate by placing the DAE triangle centroids on
the STL ones through a spatial hash at 0.2 mm and accepting only a transform
that matches every sampled triangle. It is idempotent and re-runnable when the
CAD is exported again.

The tool mount needed more than a reframe. Its visual, part61.stl, was an
export of the part rotated 45.05 degrees about y, which is what made the pen
look bolted on askew. part6.stl in the same CAD drop is the identical mesh
correctly oriented: same 5094 triangles, same 61.99 cm2, bounding boxes
matching to 0.01 mm after the rotation is undone. That export is now the tool
mount, and the duplicate pair is gone.

With the bracket square, the servo axis can be stated rather than inferred:
the clamp faces sit 12.0 mm apart around x = 5 mm and the part is symmetric
about z = 0, so tool0 moves onto that line where it leaves the outer face.

File: src/tattotronix_description/urdf/arm_macro.xacro (robot description, xacro)
@@ -112,12 +112,13 @@
     </joint>
     <!-- Tool mount: a bracket carrying a continuous-rotation SG90.
-         The mesh is a clamp whose two arms face each other across a 12.0 mm
-         gap, which is the body width of an SG90, so the servo sits between
-         them with its output shaft on the bracket's y axis. What that servo
-         ends up driving is not settled, so nothing here actuates: the tool
-         attaches through a fixed joint and the axis is recorded, not moved. -->
+         Two clamp arms face each other across a 12.0 mm gap, the body width of
+         an SG90, so the servo sits between them with its output shaft on the
+         bracket's y axis. The mesh is symmetric about z = 0, which puts that
+         shaft on the z = 0 plane. What the servo drives is not settled, so
+         nothing here actuates: the tool attaches through a fixed joint and the
+         axis is recorded, not moved. -->
     <xacro:tattotronix_link name="tool_mount_link" mass="0.15"
-        cx="0.0076" cy="-0.01155" cz="-0.0037"
-        sx="0.0492" sy="0.0231" sz="0.0414"/>
+        cx="0.0108" cy="-0.0115" cz="0.0"
+        sx="0.0365" sy="0.0231" sz="0.0330"/>
     <!-- tool flange.
          tool0 is the frame every end effector attaches to, and its +z axis is
@@ -125,9 +126,7 @@
          It is placed on the servo axis rather than guessed: the bracket's two
          clamp faces lie at y = -6.0 mm and y = -18.0 mm and share a centroid
-         at x = 4.5 mm, z = -3.0 mm, which fixes the shaft line. tool0 sits
-         where that line leaves the outer face of the bracket, y = -23.1 mm,
-         with +z pointing away from the arm. This is why the pen used to look
-         wrong: it was mounted along +x, across the servo shaft instead of
-         along it.
+         near x = 5 mm, and the part is symmetric about z = 0, which fixes the
+         shaft line. tool0 sits where that line leaves the outer face of the
+         bracket, y = -23.1 mm, with +z pointing away from the arm.
          Read off the mesh, not off CAD datums. Expect it to move by a
          millimetre or two once the bracket is measured. -->
@@ -135,5 +134,5 @@
       <parent link="tool_mount_link"/>
       <child link="tool0"/>
-      <origin xyz="0.0045 -0.0231 -0.0030" rpy="${pi/2} 0 0"/>
+      <origin xyz="0.005 -0.0231 0" rpy="${pi/2} 0 0"/>
     </joint>
     <link name="tool0"/>

Commit message: Mount the pen on the bracket tab instead of in mid air
tool0 sat at x = 5 mm on the bracket's outer face, taken from the centroid of
the clamp arms. There is no bracket there. The clamp arms stop at y = -18.0 mm
and the only material that reaches the outer face at y = -23.1 mm is a tab
spanning x = 26.0 to 29.0 mm, z = -3.6 to 14.6 mm, so the pen was growing out
of empty space beside the part.

tool0 moves to the centre of that tab, the one place on that face a tool has
anything to bolt to.

The tab is 3 mm thick and 18 mm long, which is a fixing point and not a shaft
boss, so this is where a pen would attach rather than where the servo drives
it. That distinction stops mattering once the pen itself is built.

File: src/tattotronix_description/urdf/arm_macro.xacro (robot description, xacro)
@@ -124,15 +124,16 @@
          tool0 is the frame every end effector attaches to, and its +z axis is
          the tool axis, so a tool mounts with no rotation of its own.
-         It is placed on the servo axis rather than guessed: the bracket's two
-         clamp faces lie at y = -6.0 mm and y = -18.0 mm and share a centroid
-         near x = 5 mm, and the part is symmetric about z = 0, which fixes the
-         shaft line. tool0 sits where that line leaves the outer face of the
-         bracket, y = -23.1 mm, with +z pointing away from the arm.
-         Read off the mesh, not off CAD datums. Expect it to move by a
-         millimetre or two once the bracket is measured. -->
+         Its position is measured off the bracket. The clamp arms end at
+         y = -18.0 mm and the only material beyond them, on the outer face, is
+         a tab spanning x = 26.0 to 29.0 mm and z = -3.6 to 14.6 mm, reaching
+         y = -23.1 mm. tool0 sits at the centre of that tab with +z pointing
+         away from the arm, which is the one place on that face a tool has
+         anything to bolt to.
+         Read off the mesh, not off CAD datums, and the pen the tab actually
+         carries has not been built yet. Expect this to move once it is. -->
     <joint name="tool_mount_to_tool0" type="fixed">
       <parent link="tool_mount_link"/>
       <child link="tool0"/>
-      <origin xyz="0.005 -0.0231 0" rpy="${pi/2} 0 0"/>
+      <origin xyz="0.0275 -0.0231 0.0055" rpy="${pi/2} 0 0"/>
     </joint>
     <link name="tool0"/>
