Commit message: Put the tool axis on the servo bore instead of the bracket tab
tool0 sat at the centroid of the outer tab, y = -23.1 mm, which is a fixing
feature: a 3 mm plate with nothing turned about it. A tool hung there is
bolted to the bracket but not aligned to anything that rotates, so every
tattoo path would have been planned about a line the hardware does not drive.

The bracket carries two sets of three holes and the previous reading took the
wrong set. The holes bored along y, radius 1.50 mm at x = 0 and z = -8, 0 and
+8 mm, pass through the 3 mm back plate and are how the bracket bolts down.
The holes bored along x through the outer face are the working set: radius
1.50 mm on a straight line at 8.00 mm pitch, centres at (-5.203, +9.603),
(-12.064, +5.489) and (-18.925, +1.375) in mm.

tool0 moves to the middle of that line, y = -12.064 mm, z = +5.489 mm, and
its axis becomes the bracket's own +x. Three independent measurements off the
mesh agree on it:

  * the through hole itself fits a circle of radius 1.500 mm to 3 um;
  * behind it the face opens into a stepped boss of radius 2.50, 3.00 and
    4.00 mm running back to x = 21.5 mm, and all four cylinders are
    concentric to within 5 um, which is a bearing seat and not a bolt hole;
  * the point lies on the clamp mid plane, y = -12.06 mm, and on the midpoint
    of its two neighbours to within 0.1 um.

x stays on the outer face at 29.0 mm so the tool still starts where the part
ends. The comment on tool_mount_link is corrected with it: the shaft is not
on the z = 0 symmetry plane, and the mid plane of the clamp gap is what every
turned feature at that end of the bracket is centred on.

The link macro gains a material parameter so the bracket can be rendered as
hardware rather than as printed structure.

File: src/tattotronix_description/urdf/arm_macro.xacro (robot description, xacro)
@@ -24,5 +24,5 @@
   <xacro:property name="joint_damping" value="0.5"/>
   <xacro:property name="joint_friction" value="0.1"/>
-  <xacro:macro name="tattotronix_link" params="name mass cx cy cz sx sy sz">
+  <xacro:macro name="tattotronix_link" params="name mass cx cy cz sx sy sz material:=tattotronix_shell">
     <link name="${name}">
       <visual>
@@ -31,5 +31,5 @@
           <mesh filename="${mesh_path}/visual/${name}.stl" scale="${mesh_scale}"/>
         </geometry>
-        <material name="tattotronix_graphite"/>
+        <material name="${material}"/>
       </visual>
       <collision>
@@ -113,10 +113,11 @@
     <!-- Tool mount: a bracket carrying a continuous-rotation SG90.
          Two clamp arms face each other across a 12.0 mm gap, the body width of
-         an SG90, so the servo sits between them with its output shaft on the
-         bracket's y axis. The mesh is symmetric about z = 0, which puts that
-         shaft on the z = 0 plane. What the servo drives is not settled, so
+         an SG90, so the servo sits between them. Their common mid plane is
+         y = -12.06 mm, and every turned feature at the far end of the bracket
+         is centred on it. What the servo drives is not settled, so
          nothing here actuates: the tool attaches through a fixed joint and the
          axis is recorded, not moved. -->
     <xacro:tattotronix_link name="tool_mount_link" mass="0.15"
+        material="tattotronix_steel"
         cx="0.0108" cy="-0.0115" cz="0.0"
         sx="0.0365" sy="0.0231" sz="0.0330"/>
@@ -124,16 +125,27 @@
          tool0 is the frame every end effector attaches to, and its +z axis is
          the tool axis, so a tool mounts with no rotation of its own.
-         Its position is measured off the bracket. The clamp arms end at
-         y = -18.0 mm and the only material beyond them, on the outer face, is
-         a tab spanning x = 26.0 to 29.0 mm and z = -3.6 to 14.6 mm, reaching
-         y = -23.1 mm. tool0 sits at the centre of that tab with +z pointing
-         away from the arm, which is the one place on that face a tool has
-         anything to bolt to.
-         Read off the mesh, not off CAD datums, and the pen the tab actually
-         carries has not been built yet. Expect this to move once it is. -->
+         The tool axis is the bracket's own +x, and the line it runs along is
+         the middle of the three holes on the outer face, measured off the
+         mesh:
+           y = -12.064 mm, z = +5.489 mm
+         The bracket has two sets of three holes and they are easy to confuse.
+         The set bored along y, radius 1.50 mm at x = 0 and z = -8, 0 and
+         +8 mm, goes through the 3 mm back plate: that is how the bracket bolts
+         down, and it carries nothing. The set that matters is bored along x
+         through the outer face, radius 1.50 mm, on a straight line at 8.00 mm
+         pitch: (-5.203, +9.603), (-12.064, +5.489), (-18.925, +1.375).
+         The middle one is the shaft. Behind it the face opens into a stepped
+         boss of radius 2.50, 3.00 and 4.00 mm running back to x = 21.5 mm, all
+         four cylinders concentric to within 5 um, which is a bearing seat and
+         not a bolt hole. It also sits on the clamp mid plane, y = -12.06 mm,
+         and on the midpoint of its two neighbours. Three independent readings
+         of the same line.
+         x = 29.0 mm puts the origin on that outer face, so the tool starts
+         where the part ends.
+         Read off the mesh, not off CAD datums. -->
     <joint name="tool_mount_to_tool0" type="fixed">
       <parent link="tool_mount_link"/>
       <child link="tool0"/>
-      <origin xyz="0.0275 -0.0231 0.0055" rpy="${pi/2} 0 0"/>
+      <origin xyz="0.029 -0.012064 0.005489" rpy="0 ${pi/2} 0"/>
     </joint>
     <link name="tool0"/>

Commit message: Let the description choose its mass model, defaulting to the box
tattotronix.urdf.xacro takes mass_model:=box|printed. box is the solid-box
approximation every published number was computed with, and it stays the
default. printed is the arm as built, from the generated inertials. Only the
inertial blocks change between the two; geometry and kinematics are
identical, and a test strips the inertials from both expansions and requires
what is left to match element for element.

The default did not move. The expansions for hardware none, mock and gz were
saved before the change and compared after it, parsed, element by element:
identical. The only textual difference is the new argument's documentation,
which xacro copies into the header as a comment.

An unknown model now stops the build. Before the check, mass_model:=bogus
matched neither branch in arm_macro and gave every arm link no inertial at
all - a massless robot, which Gazebo would have loaded without a word. It now
fails with the name of the argument and the value it was given.

dynamics.load() takes the model too, so the two can be compared side by side;
left unset it follows the description's default.

File: src/tattotronix_description/urdf/arm_macro.xacro (robot description, xacro)
@@ -39,7 +39,14 @@
         </geometry>
       </collision>
-      <xacro:inertial_box mass="${mass}" x="${sx}" y="${sy}" z="${sz}">
-        <origin xyz="${cx} ${cy} ${cz}" rpy="0 0 0"/>
-      </xacro:inertial_box>
+      <!-- mass_model is set in tattotronix.urdf.xacro. The box arguments are
+           still passed either way, so the default model is untouched. -->
+      <xacro:if value="${mass_model == 'printed'}">
+        <xacro:call macro="printed_inertial_${name}"/>
+      </xacro:if>
+      <xacro:if value="${mass_model == 'box'}">
+        <xacro:inertial_box mass="${mass}" x="${sx}" y="${sy}" z="${sz}">
+          <origin xyz="${cx} ${cy} ${cz}" rpy="0 0 0"/>
+        </xacro:inertial_box>
+      </xacro:if>
     </link>
   </xacro:macro>

File: src/tattotronix_description/urdf/tattotronix.urdf.xacro (robot description, xacro)
@@ -21,4 +21,11 @@
                         arm is anchored in simulation. Set false when the
                         description is embedded in a larger cell.
+      mass_model        box (default) approximates each link by the solid box
+                        that fits its bounding box, with masses written by hand.
+                        printed is the arm as built: each link's printed shell,
+                        integrated from its mesh, plus the servos mounted in it,
+                        generated into inertials_printed.xacro by
+                        docs/scripts/mass_properties.py. Only inertia changes;
+                        geometry and kinematics are identical in both.
   -->
   <xacro:arg name="hardware" default="none"/>
@@ -26,8 +33,17 @@
   <xacro:arg name="controllers_file" default=""/>
   <xacro:arg name="use_world_link" default="true"/>
+  <xacro:arg name="mass_model" default="box"/>
   <xacro:property name="hardware" value="$(arg hardware)"/>
   <xacro:property name="tool" value="$(arg tool)"/>
   <xacro:property name="use_world_link" value="$(arg use_world_link)"/>
+  <xacro:property name="mass_model" value="$(arg mass_model)"/>
+  <!-- An unknown model would otherwise match neither branch in arm_macro and
+       leave every arm link with no inertial at all: a massless robot that
+       Gazebo loads without a word. -->
+  <xacro:if value="${mass_model not in ['box', 'printed']}">
+    ${xacro.fatal('mass_model must be box or printed, not ' + str(mass_model))}
+  </xacro:if>
   <xacro:include filename="$(find tattotronix_description)/urdf/materials.xacro"/>
+  <xacro:include filename="$(find tattotronix_description)/urdf/inertials_printed.xacro"/>
   <xacro:include filename="$(find tattotronix_description)/urdf/arm_macro.xacro"/>
   <xacro:include filename="$(find tattotronix_description)/urdf/tattoo_tool.xacro"/>

Commit message: Add the second SG90, the one that drives the tool
The built arm has five large servos and two SG90s, not one. The builder
confirmed it: one SG90 turns joint_5, and a second, continuous-rotation one
drives the tool. That second one is the servo the tool mount was designed
around - its two clamp arms stand 12.0 mm apart, an SG90's body width, as
measured off the bracket mesh - and the model had left it out. It weighs 9 g
on a link whose printed shell weighs 4.6 g, so the omission nearly tripled
the error on the last link's mass.

It now sits on the tool axis. Two of its three coordinates are measurements
the description already records - the axis runs at y = -12.064 mm,
z = +5.489 mm, tool0's origin and the clamp's mid plane - and they are read
from the tool_mount_to_tool0 joint rather than written again. The third, how
far along the bracket the body sits, is not measured; it is taken as the
bracket's centroid, since the servo fills the space between the clamp arms.

That declaration was measured rather than trusted. Moving the servo 5 mm
either way changes the link's own inertia about joint_5 by -20 to +36%,
which is not small. But joint_5 is dominated by the pen, and what reaches
the gains - the effective inertia of each joint at the tuning pose - moves by
1.0 to 3.4%, most at joints 5 and 3. A test holds it under 5%.

The inventory itself is tested: five large, two small, every joint driven,
and the tool servo on the measured axis. The description's comment on the
tool mount no longer says what the servo drives is unsettled.

The description's default is still the box model, so no published number
moves here. The switch is the next step.

File: src/tattotronix_description/urdf/arm_macro.xacro (robot description, xacro)
@@ -122,7 +122,9 @@
          an SG90, so the servo sits between them. Their common mid plane is
          y = -12.06 mm, and every turned feature at the far end of the bracket
-         is centred on it. What the servo drives is not settled, so
-         nothing here actuates: the tool attaches through a fixed joint and the
-         axis is recorded, not moved. -->
+         is centred on it. The servo drives the tool, not the arm: it is one of
+         two SG90s on the built arm, the other turning joint_5. Nothing here
+         actuates it - the tool attaches through a fixed joint and the axis is
+         recorded, not moved - but its 9 g is in the printed mass model, on
+         the tool axis. -->
     <xacro:tattotronix_link name="tool_mount_link" mass="0.15"
         material="tattotronix_steel"

File: src/tattotronix_description/urdf/inertials_printed.xacro (robot description, xacro)
@@ -7,5 +7,6 @@
   Each link is its printed shell - the mesh volume at 434 kg/m^3, which is
   35% of solid PLA - plus the servos mounted in it, each a box of
-  catalogue size at the origin of the joint it drives. The volumes are
+  catalogue size at the origin of the joint it drives, or on the tool
+  axis for the one that drives the tool. The volumes are
   measured. The printed fraction and the servo figures are declarations
   about an arm that cannot be weighed, and are named in the script.
@@ -59,11 +60,11 @@
     </inertial>
   </xacro:macro>
-  <!-- tool_mount_link: shell 0.0046 kg, no servo -->
+  <!-- tool_mount_link: shell 0.0046 kg, SG90 driving the tool -->
   <xacro:macro name="printed_inertial_tool_mount_link">
     <inertial>
-      <origin xyz="0.008634 -0.010107 0.000914" rpy="0 0 0"/>
-      <mass value="0.00464284592"/>
-      <inertia ixx="4.141313e-07" ixy="5.591683e-08" ixz="-6.548634e-08"
-               iyy="6.964300e-07" iyz="6.213871e-09" izz="5.366602e-07"/>
+      <origin xyz="0.008634 -0.011398 0.003932" rpy="0 0 0"/>
+      <mass value="0.0136428459"/>
+      <inertia ixx="9.808574e-07" ixy="5.591683e-08" ixz="-6.548634e-08"
+               iyy="1.526682e-06" iyz="3.363561e-08" izz="1.032509e-06"/>
     </inertial>
   </xacro:macro>
