Commit message: Describe the real arm: a pca9685 backend with its servo calibration
tattotronix.urdf.xacro gains hardware:=pca9685. It loads the driver added in
the previous commit, and gives each joint its channel and calibration from
config/servo_calibration.yaml, which the description now installs:

- the calibration is declared, not measured, and says so: every servo is the
  catalogue convention, 1500 us at mid travel and 636.62 us per radian;
- the shoulder's second servo is declared as mounted facing the first, with a
  negative scale, and the file says what happens if that is wrong;
- the real arm's joints have no effort state, since a hobby servo reports
  nothing and the driver refuses to invent one;
- the arguments i2c_device, i2c_address, dry_run and servo_calibration reach
  it from the command line.

An unknown backend now stops the expansion, as an unknown mass model already
did, instead of giving ros2_control a system with no hardware in it. MoveIt
accepts pca9685 so it can plan from a PC against the real arm.

tests/test_hardware_description.py expands the description with every
backend and reads the result back: every servo in the calibration reaches its
joint with every parameter, no two share a channel, the real arm asks for no
effort, and the other backends keep theirs. The notebooks' expanded URDFs are
regenerated; only their comments change.

File: src/tattotronix_description/urdf/tattotronix.ros2_control.xacro (robot description, xacro)
@@ -7,9 +7,16 @@
       mock  -> mock_components/GenericSystem, for testing controllers and
                MoveIt with no simulator and no hardware attached
-    The real driver is not written yet. The launch files validate the argument
-    before they call xacro, so an unknown backend is rejected there rather than
-    producing a description that silently controls nothing.
+      pca9685 -> tattotronix_hardware/Pca9685ServoSystem, the arm as built:
+               hobby servos driven through a PCA9685 board. Each joint gets
+               its channel and calibration from servo_calibration.
+    tattotronix.urdf.xacro rejects any other backend, so an unknown one fails
+    at expansion rather than producing a description that controls nothing.
+    The pca9685 joints have no effort state. A hobby servo reports nothing, so
+    the driver refuses to invent one, and its position and velocity states are
+    the command it last sent rather than a measurement.
   -->
-  <xacro:macro name="tattotronix_ros2_control" params="name hardware">
+  <xacro:macro name="tattotronix_ros2_control"
+               params="name hardware i2c_device:=/dev/i2c-1 i2c_address:=64 dry_run:=false
+                       servo_calibration:=''">
     <ros2_control name="${name}" type="system">
       <xacro:if value="${hardware == 'gz'}">
@@ -25,4 +32,15 @@
         </hardware>
       </xacro:if>
+      <xacro:if value="${hardware == 'pca9685'}">
+        <xacro:property name="calibration" value="${xacro.load_yaml(servo_calibration)}"/>
+        <hardware>
+          <plugin>tattotronix_hardware/Pca9685ServoSystem</plugin>
+          <param name="i2c_device">${i2c_device}</param>
+          <param name="i2c_address">${i2c_address}</param>
+          <param name="frame_rate_hz">50</param>
+          <param name="oscillator_hz">25000000</param>
+          <param name="dry_run">${dry_run}</param>
+        </hardware>
+      </xacro:if>
       <xacro:macro name="controlled_joint" params="name initial_position">
         <joint name="${name}">
@@ -35,5 +53,20 @@
           </state_interface>
           <state_interface name="velocity"/>
-          <state_interface name="effort"/>
+          <xacro:unless value="${hardware == 'pca9685'}">
+            <state_interface name="effort"/>
+          </xacro:unless>
+          <xacro:if value="${hardware == 'pca9685'}">
+            <xacro:property name="servo" value="${calibration['servos'][name]}"/>
+            <param name="channel">${servo['channel']}</param>
+            <param name="zero_us">${servo['zero_us']}</param>
+            <param name="us_per_rad">${servo['us_per_rad']}</param>
+            <param name="min_us">${servo['min_us']}</param>
+            <param name="max_us">${servo['max_us']}</param>
+            <xacro:if value="${'channel_b' in servo}">
+              <param name="channel_b">${servo['channel_b']}</param>
+              <param name="zero_us_b">${servo['zero_us_b']}</param>
+              <param name="us_per_rad_b">${servo['us_per_rad_b']}</param>
+            </xacro:if>
+          </xacro:if>
         </joint>
       </xacro:macro>

File: src/tattotronix_description/urdf/tattotronix.urdf.xacro (robot description, xacro)
@@ -6,8 +6,18 @@
     Swap the tool argument and the same arm carries a different end effector.
     Arguments
-      hardware          gz | mock | none
+      hardware          gz | mock | pca9685 | none
                         'none' leaves ros2_control out entirely, which is what
                         display.launch.py wants: a description RViz can render
                         with joint_state_publisher_gui and no controller stack.
+                        'pca9685' is the arm as built: its hobby servos driven
+                        through a PCA9685 board by tattotronix_hardware.
+      i2c_device        pca9685 only: the Linux I2C bus the board is on.
+      i2c_address       pca9685 only: the board's address; 64 is 0x40, the
+                        address with no jumpers soldered.
+      dry_run           pca9685 only: true runs the whole stack with the board
+                        simulated, sending nothing. For a first run, and for CI.
+      servo_calibration pca9685 only: which channel drives each joint and how
+                        its pulse maps to the angle. The default is declared,
+                        not measured; see config/servo_calibration.yaml.
       tool              tattoo | none
                         The pen in tattoo_tool.xacro is primitives sized to a
@@ -36,4 +46,9 @@
   <xacro:arg name="use_world_link" default="true"/>
   <xacro:arg name="mass_model" default="printed"/>
+  <xacro:arg name="i2c_device" default="/dev/i2c-1"/>
+  <xacro:arg name="i2c_address" default="64"/>
+  <xacro:arg name="dry_run" default="false"/>
+  <xacro:arg name="servo_calibration"
+             default="$(find tattotronix_description)/config/servo_calibration.yaml"/>
   <xacro:property name="hardware" value="$(arg hardware)"/>
   <xacro:property name="tool" value="$(arg tool)"/>
@@ -45,4 +60,10 @@
   <xacro:if value="${mass_model not in ['box', 'printed']}">
     ${xacro.fatal('mass_model must be box or printed, not ' + str(mass_model))}
+  </xacro:if>
+  <!-- The same for the backend: an unknown one would match no branch in the
+       ros2_control macro and give the controller manager a system with no
+       hardware in it. -->
+  <xacro:if value="${hardware not in ['gz', 'mock', 'pca9685', 'none']}">
+    ${xacro.fatal('hardware must be gz, mock, pca9685 or none, not ' + str(hardware))}
   </xacro:if>
   <xacro:include filename="$(find tattotronix_description)/urdf/materials.xacro"/>
@@ -72,5 +93,7 @@
   </xacro:if>
   <xacro:unless value="${hardware == 'none'}">
-    <xacro:tattotronix_ros2_control name="tattotronix_system" hardware="${hardware}"/>
+    <xacro:tattotronix_ros2_control name="tattotronix_system" hardware="${hardware}"
+      i2c_device="$(arg i2c_device)" i2c_address="$(arg i2c_address)"
+      dry_run="$(arg dry_run)" servo_calibration="$(arg servo_calibration)"/>
   </xacro:unless>
   <xacro:if value="${hardware == 'gz'}">

Commit message: Drive the tool's continuous servo as a speed, on the real arm
The tool's continuous-rotation SG90 turns a pulse into a speed, not an angle,
so it is not a joint. The driver now takes it as a gpio with a speed interface
from -1 to 1: stop_us is the pulse at which it stands still, us_per_speed the
pulse added for full speed, both declared in the calibration like the rest.
A speed of zero sends no pulse at all, because the stopping pulse is a trim
that drifts and no pulse always stops the servo; the channel is off when the
driver activates, and anything past full speed is held to it.

The description gives the real arm the tool once the calibration names its
stop pulse, on a channel of its own. config/hardware.yaml adds tool_controller,
a forward_command_controller on that interface, which only the real arm has,
and keeps the tool out of /joint_states, where robot_state_publisher and MoveIt
read the arm's joints. arm.launch.py spawns it.

Tests: the driver keeps the tool off until it is asked to turn, sends the
right pulse for half speed, never passes full speed, switches off again at
zero, and refuses a tool on a joint's channel; the description carries the
tool's calibration to the driver; and the dry run brings tool_controller up
with the rest and checks /joint_states names the five joints and nothing else.

File: src/tattotronix_description/urdf/tattotronix.ros2_control.xacro (robot description, xacro)
@@ -76,4 +76,22 @@
       <xacro:controlled_joint name="joint_4" initial_position="0.0"/>
       <xacro:controlled_joint name="joint_5" initial_position="0.0"/>
+      <!-- The tool's continuous servo, on the real arm, once the calibration
+           gives its stop pulse. A speed rather than an angle, so a gpio
+           rather than a joint, and nothing robot_state_publisher needs. -->
+      <xacro:if value="${hardware == 'pca9685' and 'tool' in calibration and 'stop_us' in calibration['tool']}">
+        <xacro:property name="tool_servo" value="${calibration['tool']}"/>
+        <gpio name="tool">
+          <command_interface name="speed">
+            <param name="min">-1</param>
+            <param name="max">1</param>
+          </command_interface>
+          <state_interface name="speed"/>
+          <param name="channel">${tool_servo['channel']}</param>
+          <param name="stop_us">${tool_servo['stop_us']}</param>
+          <param name="us_per_speed">${tool_servo['us_per_speed']}</param>
+          <param name="min_us">${tool_servo['min_us']}</param>
+          <param name="max_us">${tool_servo['max_us']}</param>
+        </gpio>
+      </xacro:if>
     </ros2_control>
   </xacro:macro>

Commit message: Revert driving the tool-mount servo: it is a leftover, not a tool
This reverts commit e5573ba.

The continuous SG90 clamped in the tool mount was put there for a gripper the
arm was first designed to carry. The arm draws instead, and the owner has said
the tip must not turn: that servo drives nothing. So the driver no longer
takes it as a speed interface, the description no longer gives it one, and
tool_controller, its spawner and its dependency on forward_command_controller
go with them.

The tree is back to c28e46e byte for byte, which is the tree the full test
suite last certified. The places that still describe that servo as driving the
tool are corrected in the next commit.

File: src/tattotronix_description/urdf/tattotronix.ros2_control.xacro (robot description, xacro)
@@ -76,22 +76,4 @@
       <xacro:controlled_joint name="joint_4" initial_position="0.0"/>
       <xacro:controlled_joint name="joint_5" initial_position="0.0"/>
-      <!-- The tool's continuous servo, on the real arm, once the calibration
-           gives its stop pulse. A speed rather than an angle, so a gpio
-           rather than a joint, and nothing robot_state_publisher needs. -->
-      <xacro:if value="${hardware == 'pca9685' and 'tool' in calibration and 'stop_us' in calibration['tool']}">
-        <xacro:property name="tool_servo" value="${calibration['tool']}"/>
-        <gpio name="tool">
-          <command_interface name="speed">
-            <param name="min">-1</param>
-            <param name="max">1</param>
-          </command_interface>
-          <state_interface name="speed"/>
-          <param name="channel">${tool_servo['channel']}</param>
-          <param name="stop_us">${tool_servo['stop_us']}</param>
-          <param name="us_per_speed">${tool_servo['us_per_speed']}</param>
-          <param name="min_us">${tool_servo['min_us']}</param>
-          <param name="max_us">${tool_servo['max_us']}</param>
-        </gpio>
-      </xacro:if>
     </ros2_control>
   </xacro:macro>
